File: Hardware/Triple_Axis_Accelerometer_-_Gyro_Breakout_-_MPU-6050.brd (EAGLE design)
At the start: 25.4 x 15.2 mm, 20 parts, among them U1 MPU-6050-1, U3 CREATIVE_COMMONS

Commit message: Fixed formatting issues on schematic and board file
Parts:
- removed U3: CREATIVE_COMMONS, SparkFun:CREATIVE_COMMONS
- added FRAME1: FRAME-LETTER, SparkFun-Aesthetics:CREATIVE_COMMONS
- added U$5: REVISION, SparkFun-Aesthetics:REVISION
Other:
- board text added: "Eric Orosel"
